File: PCB/keyboard.kicad_pcb (KiCad board)
At the start: 2 copper layers, 319.3 x 100.2 mm, 153 parts, among them J1 USB_C_Receptacle_USB2.0, SW1 SW_Push, SW10 SW_Push, SW11 SW_Push, SW12 SW_Push, SW13 SW_Push, SW14 SW_Push, SW15 SW_Push, SW16 SW_Push, SW17 SW_Push, SW18 SW_Push, SW19 SW_Push, SW2 SW_Push, SW20 SW_Push, SW21 SW_Push, SW22 SW_Push, SW23 SW_Push, SW24 SW_Push, SW25 SW_Push, SW26 SW_Push, SW27 SW_Push, SW28 SW_Push, SW29 SW_Push, SW3 SW_Push, SW30 SW_Push, SW31 SW_Push, SW32 SW_Push, SW33 SW_Push, SW34 SW_Push, SW35 SW_Push, SW36 SW_Push, SW37 SW_Push, SW38 SW_Push, SW39 SW_Push, SW4 SW_Push, SW40 SW_Push, SW41 SW_Push, SW42 SW_Push, SW43 SW_Push, SW44 SW_Push, SW45 SW_Push, SW46 SW_Push, SW47 SW_Push, SW48 SW_Push, SW49 SW_Push, SW5 SW_Push, SW50 SW_Push, SW51 SW_Push, SW52 SW_Push, SW53 SW_Push, SW54 SW_Push, SW55 SW_Push, SW56 SW_Push, SW57 SW_Push, SW58 SW_Push, SW59 SW_Push, SW6 SW_Push, SW60 SW_Push, SW61 SW_Push, SW62 SW_Push, SW63 SW_Push, SW64 SW_Push, SW65 SW_Push, SW66 SW_Push, SW67 SW_Push, SW68 SW_Push, SW7 SW_Push, SW8 SW_Push, SW9 SW_Push, U1 ATmega16U4-AU, U2 TPD2S017, Y1 Crystal_GND24

Commit message: configured footprints
Connections:
- net mcu/~HWB~/PE2 renamed mcu/~{HWB}/PE2
- net mcu/~RESET renamed mcu/~{RESET}
Routing:
- net (no net): track 1777.1 -> 0.00 mm
- net COL10: track 0.00 -> 89.0 mm
- net COL12: track 0.00 -> 87.0 mm
- net COL6: track 0.00 -> 87.0 mm
- net COL2: track 0.00 -> 87.0 mm
- net COL11: track 0.00 -> 87.0 mm
- net COL1: track 0.00 -> 84.1 mm
- net COL0: track 0.00 -> 81.1 mm
- net COL14: track 0.00 -> 80.1 mm
- net COL16: track 0.00 -> 76.2 mm
- net COL9: track 0.00 -> 67.0 mm
- net COL8: track 0.00 -> 67.0 mm
- net COL5: track 0.00 -> 67.0 mm
- net COL7: track 0.00 -> 67.0 mm
- net COL4: track 0.00 -> 67.0 mm
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Other:
- net class Default removed

Commit message: Started pcb development
Parts:
- removed C8: 1u, C_0603_1608Metric
- removed J1: USB_C_Receptacle_USB2.0, USB_C_Receptacle_XKB_U262-16XN-4BVC11
- removed RST: SW_SPST, SW_SPST_TL3342
- removed SW10, SW11, SW12, SW13, SW15, SW17, SW18, SW19, SW2, SW20, SW21, SW22, SW23, SW24, SW25, SW26, SW27, SW28, SW3, SW30, SW32, SW33, SW34, SW35, SW36, SW37, SW38, SW39, SW4, SW40, SW41, SW42, SW44, SW46, SW47, SW48, SW49, SW5, SW50, SW51, SW52, SW53, SW54, SW55, SW57, SW58, SW6, SW60, SW66, SW67, SW68, SW7, SW8, SW9: SW_Push, MX-1U-NoLED
- removed SW14: SW_Push, MX-2U-NoLED
- removed SW16, SW29: SW_Push, MX-1.5U-NoLED
- removed SW31: SW_Push, MX-1.75U-NoLED
- removed SW43, SW45, SW56: SW_Push, MX-2.25U-NoLED
- removed SW59, SW61, SW63, SW64, SW65: SW_Push, MX-1.25U-NoLED
- removed SW62: SW_Push, MX-6.25U-NoLED
- removed U2: TPD2S017, SOT-23-6
- added F1: 500mA, Fuse:Fuse_1206_3216Metric, F.Cu at (283.1, 45.6)
- added MX1: MX-NoLED, MX_Alps_Hybrid:MX-1U-NoLED, F.Cu at (189.4, 108.0)
- added MX10: MX-NoLED, MX_Alps_Hybrid:MX-1U-NoLED, F.Cu at (209.6, 47.4)
- added MX11: MX-NoLED, MX_Alps_Hybrid:MX-1U-NoLED, F.Cu at (169.2, 87.8)
- added MX12: MX-NoLED, MX_Alps_Hybrid:MX-1U-NoLED, F.Cu at (270.2, 47.4)
- added MX13: MX-NoLED, MX_Alps_Hybrid:MX-1U-NoLED, F.Cu at (149.0, 128.2)
- added MX14: MX-NoLED, MX_Alps_Hybrid:MX-1U-NoLED, F.Cu at (88.4, 47.4)
- added MX15: MX-NoLED, MX_Alps_Hybrid:MX-1U-NoLED, F.Cu at (108.6, 47.4)
- added MX16: MX-NoLED, MX_Alps_Hybrid:MX-1U-NoLED, F.Cu at (209.6, 67.6)
- added MX17: MX-NoLED, MX_Alps_Hybrid:MX-1U-NoLED, F.Cu at (169.2, 47.4)
- added MX18: MX-NoLED, MX_Alps_Hybrid:MX-1U-NoLED, F.Cu at (68.2, 47.4)
- added MX19: MX-NoLED, MX_Alps_Hybrid:MX-1U-NoLED, F.Cu at (48.0, 108.0)
- added MX2: MX-NoLED, MX_Alps_Hybrid:MX-1U-NoLED, F.Cu at (128.8, 128.2)
- added MX20: MX-NoLED, MX_Alps_Hybrid:MX-1U-NoLED, F.Cu at (68.2, 148.4)
- added MX21: MX-NoLED, MX_Alps_Hybrid:MX-1U-NoLED, F.Cu at (48.0, 47.4)
- added MX22: MX-NoLED, MX_Alps_Hybrid:MX-1U-NoLED, F.Cu at (108.6, 108.0)
- added MX23: MX-NoLED, MX_Alps_Hybrid:MX-1U-NoLED, F.Cu at (250.0, 67.6)
- added MX24: MX-NoLED, MX_Alps_Hybrid:MX-1U-NoLED, F.Cu at (128.8, 148.4)
- added MX25: MX-NoLED, MX_Alps_Hybrid:MX-1U-NoLED, F.Cu at (169.2, 168.6)
- added MX26: MX-NoLED, MX_Alps_Hybrid:MX-1U-NoLED, F.Cu at (189.4, 47.4)
- added MX27: MX-NoLED, MX_Alps_Hybrid:MX-1U-NoLED, F.Cu at (68.2, 67.6)
- added MX28: MX-NoLED, MX_Alps_Hybrid:MX-1U-NoLED, F.Cu at (48.0, 168.6)
- added MX29: MX-NoLED, MX_Alps_Hybrid:MX-1U-NoLED, F.Cu at (169.2, 128.2)
- added MX3: MX-NoLED, MX_Alps_Hybrid:MX-1U-NoLED, F.Cu at (169.2, 108.0)
- added MX30: MX-NoLED, MX_Alps_Hybrid:MX-1U-NoLED, F.Cu at (108.6, 128.2)
- added MX31: MX-NoLED, MX_Alps_Hybrid:MX-1U-NoLED, F.Cu at (48.0, 128.2)
- added MX32: MX-NoLED, MX_Alps_Hybrid:MX-1U-NoLED, F.Cu at (229.8, 108.0)
- added MX33: MX-NoLED, MX_Alps_Hybrid:MX-1U-NoLED, F.Cu at (250.0, 47.4)
- added MX34: MX-NoLED, MX_Alps_Hybrid:MX-1U-NoLED, F.Cu at (48.0, 67.6)
- added MX35: MX-NoLED, MX_Alps_Hybrid:MX-1U-NoLED, F.Cu at (189.4, 67.6)
- added MX36: MX-NoLED, MX_Alps_Hybrid:MX-1U-NoLED, F.Cu at (169.2, 67.6)
- added MX37: MX-NoLED, MX_Alps_Hybrid:MX-1U-NoLED, F.Cu at (209.6, 87.8)
- added MX38: MX-NoLED, MX_Alps_Hybrid:MX-1U-NoLED, F.Cu at (169.2, 148.4)
- added MX39: MX-NoLED, MX_Alps_Hybrid:MX-1U-NoLED, F.Cu at (128.8, 47.4)
- added MX4: MX-NoLED, MX_Alps_Hybrid:MX-1U-NoLED, F.Cu at (88.4, 168.6)
- added MX40: MX-NoLED, MX_Alps_Hybrid:MX-1U-NoLED, F.Cu at (88.4, 108.0)
- added MX41: MX-NoLED, MX_Alps_Hybrid:MX-1U-NoLED, F.Cu at (108.6, 67.6)
- added MX42: MX-NoLED, MX_Alps_Hybrid:MX-1U-NoLED, F.Cu at (149.0, 67.6)
- added MX43: MX-NoLED, MX_Alps_Hybrid:MX-1U-NoLED, F.Cu at (128.8, 87.8)
- added MX44: MX-NoLED, MX_Alps_Hybrid:MX-1U-NoLED, F.Cu at (88.4, 87.8)
- added MX45: MX-NoLED, MX_Alps_Hybrid:MX-1U-NoLED, F.Cu at (68.2, 108.0)
- added MX46: MX-NoLED, MX_Alps_Hybrid:MX-1U-NoLED, F.Cu at (189.4, 87.8)
- added MX47: MX-NoLED, MX_Alps_Hybrid:MX-1U-NoLED, F.Cu at (149.0, 108.0)
- added MX48: MX-NoLED, MX_Alps_Hybrid:MX-1U-NoLED, F.Cu at (68.2, 87.8)
- added MX49: MX-NoLED, MX_Alps_Hybrid:MX-1U-NoLED, F.Cu at (128.8, 168.6)
- added MX5: MX-NoLED, MX_Alps_Hybrid:MX-1U-NoLED, F.Cu at (209.6, 108.0)
- added MX50: MX-NoLED, MX_Alps_Hybrid:MX-1U-NoLED, F.Cu at (108.6, 148.4)
- added MX51: MX-NoLED, MX_Alps_Hybrid:MX-1U-NoLED, F.Cu at (229.8, 87.8)
- added MX52: MX-NoLED, MX_Alps_Hybrid:MX-1U-NoLED, F.Cu at (68.2, 128.2)
- added MX53: MX-NoLED, MX_Alps_Hybrid:MX-1U-NoLED, F.Cu at (149.0, 148.4)
- added MX54: MX-NoLED, MX_Alps_Hybrid:MX-1U-NoLED, F.Cu at (108.6, 87.8)
- added MX55: MX-NoLED, MX_Alps_Hybrid:MX-1U-NoLED, F.Cu at (149.0, 47.4)
- added MX56: MX-NoLED, MX_Alps_Hybrid:MX-1U-NoLED, F.Cu at (149.0, 87.8)
- added MX57: MX-NoLED, MX_Alps_Hybrid:MX-1U-NoLED, F.Cu at (68.2, 168.6)
- added MX58: MX-NoLED, MX_Alps_Hybrid:MX-1U-NoLED, F.Cu at (88.4, 148.4)
- added MX59: MX-NoLED, MX_Alps_Hybrid:MX-1U-NoLED, F.Cu at (189.4, 148.4)
- added MX6: MX-NoLED, MX_Alps_Hybrid:MX-1U-NoLED, F.Cu at (128.8, 67.6)
- added MX60: MX-NoLED, MX_Alps_Hybrid:MX-1U-NoLED, F.Cu at (149.0, 168.6)
- added MX61: MX-NoLED, MX_Alps_Hybrid:MX-1U-NoLED, F.Cu at (48.0, 148.4)
- added MX62: MX-NoLED, MX_Alps_Hybrid:MX-1U-NoLED, F.Cu at (128.8, 108.0)
- added MX63: MX-NoLED, MX_Alps_Hybrid:MX-1U-NoLED, F.Cu at (48.0, 87.8)
- added MX64: MX-NoLED, MX_Alps_Hybrid:MX-1U-NoLED, F.Cu at (88.4, 128.2)
- added MX65: MX-NoLED, MX_Alps_Hybrid:MX-1U-NoLED, F.Cu at (229.8, 67.6)
- added MX66: MX-NoLED, MX_Alps_Hybrid:MX-1U-NoLED, F.Cu at (250.0, 87.8)
- added MX67: MX-NoLED, MX_Alps_Hybrid:MX-1U-NoLED, F.Cu at (88.4, 67.6)
- added MX68: MX-NoLED, MX_Alps_Hybrid:MX-1U-NoLED, F.Cu at (108.6, 168.6)
- added MX7: MX-NoLED, MX_Alps_Hybrid:MX-1U-NoLED, F.Cu at (209.6, 128.2)
- added MX8: MX-NoLED, MX_Alps_Hybrid:MX-1U-NoLED, F.Cu at (189.4, 128.2)
- added MX9: MX-NoLED, MX_Alps_Hybrid:MX-1U-NoLED, F.Cu at (229.8, 47.4)
- added USB1: Molex-0548190589, random-keyboard-parts:Molex-0548190589, F.Cu at (42.3, 183.8)
- C1, C2: value 22p -> 0.1uF; footprint C_0603_1608Metric -> Capacitor_SMD:C_0805_2012Metric; moved to F.Cu
- C3, C4: value 0.1u -> 22pF; footprint C_0603_1608Metric -> Capacitor_SMD:C_0805_2012Metric; moved to F.Cu
- C5: value 0.1u -> 0.1uF; footprint C_0603_1608Metric -> Capacitor_SMD:C_0805_2012Metric; moved to F.Cu
- C6: value 0.1u -> 1uf; footprint C_0603_1608Metric -> Capacitor_SMD:C_0805_2012Metric; moved to F.Cu
- C7: value 4.7u -> 10uF; footprint C_0603_1608Metric -> Capacitor_SMD:C_0805_2012Metric; moved to F.Cu
- D1, D10, D11, D12, D13, D14, D15, D16, D17, D18, D19, D2, D20, D21, D22, D23, D24, D25, D26, D27, D28, D29, D3, D30, D31, D32, D33, D34, D35, D36, D37, D38, D39, D4, D40, D41, D42, D43, D44, D45, D46, D47, D48, D49, D5, D50, D51, D52, D53, D54, D55, D56, D57, D58, D59, D6, D60, D61, D62, D63, D64, D65, D66, D67, D68, D7, D8, D9: value D -> D_Small; footprint D_SOD-323F -> Diode_SMD:D_SOD-123; moved to F.Cu
- R1, R2, R3, R4: footprint R_0603_1608Metric -> Resistor_SMD:R_0805_2012Metric; moved to F.Cu
- SW1: footprint MX-1U-NoLED -> random-keyboard-parts:SKQG-1155865
- U1: value ATmega16U4-AU -> ATmega32U4-A; footprint TQFP-44_10x10mm_P0.8mm -> Package_QFP:TQFP-44_10x10mm_P0.8mm; moved to F.Cu
- Y1: value Crystal_GND24 -> 16MHz; footprint Crystal_SMD_3225-4Pin_3.2x2.5mm -> Crystal:Crystal_SMD_3225-4Pin_3.2x2.5mm; moved to F.Cu
- moved C7 281.0 mm to (294.1, 38.8), turned to 0 degrees
- moved C6 276.6 mm to (282.6, 51.8), turned to 0 degrees
- moved D58 275.2 mm to (74.5, 183.7), turned to 0 degrees
- moved D67 275.1 mm to (51.5, 190.0), turned to 0 degrees
- moved D30 269.3 mm to (97.5, 183.7), turned to 0 degrees
- moved C4 267.4 mm to (282.6, 48.8), turned to 0 degrees
- moved D14 265.0 mm to (80.2, 190.4), turned to 0 degrees
- moved D44 263.7 mm to (97.5, 190.4), turned to 0 degrees
- moved R4 261.1 mm to (288.2, 45.4), turned to 0 degrees
- moved D57 258.4 mm to (74.5, 187.0), turned to 0 degrees
- moved C1 257.4 mm to (287.0, 48.8), turned to 0 degrees
- moved U1 254.7 mm to (267.4, 64.7), turned to 0 degrees
- moved D59 252.6 mm to (283.2, 38.9), turned to 0 degrees
- moved C2 241.1 mm to (262.4, 73.4), turned to 0 degrees
- moved D68 241.0 mm to (103.2, 180.3), turned to 0 degrees
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Connections:
- C1 pad 1: mcu/XTAL1 -> +5V
- C2 pad 1: mcu/XTAL2 -> +5V
- C3 pad 1: VCC -> GND
- C3 pad 2: GND -> Net-(U1-XTAL1)
- C4 pad 1: VCC -> GND
- C4 pad 2: GND -> Net-(U1-XTAL2)
- C5 pad 1: VCC -> +5V
- C6 pad 1: VCC -> Net-(U1-UCAP)
- C7 pad 1: VCC -> +5V
- D1 pad 2: N$1 -> Net-(D1-A)
- D10 pad 1: ROW0 -> ROW4
- D12 pad 1: ROW0 -> ROW1
- D13 pad 1: ROW0 -> ROW2
- D14 pad 1: ROW0 -> ROW3
- D15 pad 1: ROW0 -> ROW4
- D16 pad 1: ROW1 -> ROW0
- D18 pad 1: ROW1 -> ROW2
- D19 pad 1: ROW1 -> ROW3
- D2 pad 1: ROW0 -> ROW1
- D20 pad 1: ROW1 -> ROW4
- D21 pad 1: ROW1 -> ROW0
- D23 pad 1: ROW1 -> ROW2
- D24 pad 1: ROW1 -> ROW3
- D25 pad 1: ROW1 -> ROW4
- D26 pad 1: ROW1 -> ROW0
- D28 pad 1: ROW1 -> ROW2
- D29 pad 1: ROW1 -> ROW3
- D3 pad 1: ROW0 -> ROW2
- D30 pad 1: ROW1 -> ROW4
- D31 pad 1: ROW2 -> ROW0
- D32 pad 1: ROW2 -> ROW1
- D34 pad 1: ROW2 -> ROW3
- D35 pad 1: ROW2 -> ROW4
- D36 pad 1: ROW2 -> ROW0
- D37 pad 1: ROW2 -> ROW1
- D39 pad 1: ROW2 -> ROW3
- D4 pad 1: ROW0 -> ROW3
- D40 pad 1: ROW2 -> ROW4
- D41 pad 1: ROW2 -> ROW0
- D42 pad 1: ROW2 -> ROW1
- D44 pad 1: ROW2 -> ROW3
- D45 pad 1: ROW3 -> ROW4
- D46 pad 1: ROW3 -> ROW0
- D47 pad 1: ROW3 -> ROW1
- D48 pad 1: ROW3 -> ROW2
- D5 pad 1: ROW0 -> ROW4
- D50 pad 1: ROW3 -> ROW4
- D51 pad 1: ROW3 -> ROW0
- D52 pad 1: ROW3 -> ROW1
- D53 pad 1: ROW3 -> ROW2
- D55 pad 1: ROW3 -> ROW0
- D56 pad 1: ROW3 -> ROW1
- D57 pad 1: ROW3 -> ROW2
- D59 pad 1: ROW4 -> ROW0
- D60 pad 1: ROW4 -> ROW1
- D61 pad 1: ROW4 -> ROW2
- D62 pad 1: ROW4 -> ROW3
- D63 pad 1: ROW4 -> ROW0
- D64 pad 1: ROW4 -> ROW1
- D65 pad 1: ROW4 -> ROW2
- D66 pad 1: ROW4 -> ROW3
- D67 pad 1: ROW4 -> ROW0
- D68 pad 1: ROW4 -> ROW1
- D7 pad 1: ROW0 -> ROW1
- D8 pad 1: ROW0 -> ROW2
- D9 pad 1: ROW0 -> ROW3
- R1 pad 1: mcu/D- -> D +
- R1 pad 2: u2/D- -> Net-(U1-D+)
- R2 pad 1: mcu/D+ -> D -
- R2 pad 2: u2/D+ -> Net-(U1-D-)
- R3 pad 1: mcu/~{HWB}/PE2 -> +5V
- R3 pad 2: GND -> Net-(U1-~{RESET})
- R4 pad 1: mcu/~{RESET} -> Net-(U1-~{HWB}/PE2)
- R4 pad 2: VCC -> GND
- SW1 pad 1: COL0 -> GND
- SW1 pad 2: N$1 -> Net-(U1-~{RESET})
- U1 pad 1: (no net) -> unconnected-(U1-PE6)
- U1 pad 10: ROW2 -> unconnected-(U1-PB2)
- U1 pad 11: ROW3 -> unconnected-(U1-PB3)
- U1 pad 12: COL2 -> unconnected-(U1-PB7)
- U1 pad 13: mcu/~{RESET} -> Net-(U1-~{RESET})
- U1 pad 14: VCC -> +5V
- U1 pad 16: mcu/XTAL2 -> Net-(U1-XTAL2)
- U1 pad 17: mcu/XTAL1 -> Net-(U1-XTAL1)
- U1 pad 18: COL5 -> unconnected-(U1-PD0)
- U1 pad 19: COL6 -> unconnected-(U1-PD1)
- U1 pad 2: VCC -> +5V
- U1 pad 20: COL7 -> unconnected-(U1-PD2)
- U1 pad 21: COL8 -> unconnected-(U1-PD3)
- U1 pad 22: COL10 -> unconnected-(U1-PD5)
- U1 pad 24: VCC -> +5V
- U1 pad 25: COL9 -> unconnected-(U1-PD4)
- U1 pad 26: COL11 -> unconnected-(U1-PD6)
- U1 pad 27: COL12 -> unconnected-(U1-PD7)
- U1 pad 28: ROW4 -> unconnected-(U1-PB4)
- U1 pad 29: COL0 -> unconnected-(U1-PB5)
- U1 pad 3: mcu/D- -> Net-(U1-D-)
- U1 pad 30: COL1 -> unconnected-(U1-PB6)
- U1 pad 31: COL3 -> unconnected-(U1-PC6)
- U1 pad 32: COL4 -> unconnected-(U1-PC7)
- U1 pad 33: mcu/~{HWB}/PE2 -> Net-(U1-~{HWB}/PE2)
- U1 pad 34: VCC -> +5V
- U1 pad 36: (no net) -> unconnected-(U1-PF7)
- U1 pad 37: (no net) -> unconnected-(U1-PF6)
- U1 pad 38: COL15 -> unconnected-(U1-PF5)
- U1 pad 39: COL13 -> unconnected-(U1-PF4)
- U1 pad 4: mcu/D+ -> Net-(U1-D+)
- U1 pad 40: COL16 -> unconnected-(U1-PF1)
- U1 pad 41: COL14 -> unconnected-(U1-PF0)
- U1 pad 42: (no net) -> unconnected-(U1-AREF)
- U1 pad 44: VCC -> +5V
- U1 pad 6: mcu/UCAP -> Net-(U1-UCAP)
- U1 pad 7: (no net) -> +5V
- U1 pad 8: ROW0 -> unconnected-(U1-PB0)
- U1 pad 9: ROW1 -> unconnected-(U1-PB1)
- Y1 pad 1: mcu/XTAL1 -> Net-(U1-XTAL1)
- Y1 pad 3: mcu/XTAL2 -> Net-(U1-XTAL2)
Routing:
- net ROW0: track 295.3 -> 0.00 mm
- net ROW4: track 292.9 -> 0.00 mm
- net ROW1: track 290.5 -> 0.00 mm
- net ROW2: track 288.1 -> 0.00 mm
- net ROW3: track 283.4 -> 0.00 mm
- net COL10: track 89.0 -> 0.00 mm
- net COL12: track 87.0 -> 0.00 mm
- net COL6: track 87.0 -> 0.00 mm
- net COL2: track 87.0 -> 0.00 mm
- net COL11: track 87.0 -> 0.00 mm
- net COL1: track 84.1 -> 0.00 mm
- net COL0: track 81.1 -> 0.00 mm
- net COL14: track 80.1 -> 0.00 mm
- net COL16: track 76.2 -> 0.00 mm
- net VCC: track 69.3 -> 0.00 mm
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Other:
- board outline removed

Commit message: fixed footprints
Parts:
- MX15, MX25, MX30, MX35, MX5, MX58: footprint MX_Alps_Hybrid:MX-1U-NoLED -> MX_Alps_Hybrid:MX-1.25U-NoLED
- MX2, MX64: footprint MX_Alps_Hybrid:MX-1U-NoLED -> MX_Alps_Hybrid:MX-1.5U-NoLED
- MX20: footprint MX_Alps_Hybrid:MX-1U-NoLED -> MX_Alps_Hybrid:MX-6.25U-NoLED
- MX3: footprint MX_Alps_Hybrid:MX-1U-NoLED -> MX_Alps_Hybrid:MX-1.75U-NoLED
- MX4, MX61: footprint MX_Alps_Hybrid:MX-1U-NoLED -> MX_Alps_Hybrid:MX-2.25U-NoLED
- MX63: footprint MX_Alps_Hybrid:MX-1U-NoLED -> MX_Alps_Hybrid:MX-2U-NoLED
- moved C5 302.8 mm to (316.2, 65.8)
- moved D19 265.4 mm to (316.8, 59.3)
- moved D9 263.9 mm to (316.8, 49.3)
- moved D5 259.0 mm to (322.6, 52.6)
- moved C3 252.7 mm to (280.4, 99.6)
- moved D26 240.8 mm to (316.8, 56.0)
- moved D47 240.8 mm to (322.6, 49.3)
- moved D22 238.8 mm to (286.8, 89.7)
- moved D33 237.4 mm to (281.0, 89.7)
- moved D29 235.1 mm to (328.3, 49.3)
- moved D31 228.0 mm to (306.3, 72.8)
- moved D32 226.7 mm to (291.8, 83.9)
- moved D43 218.1 mm to (306.3, 69.5)
- moved MX51 198.6 mm to (54.0, 180.2)
- moved USB1 193.8 mm to (201.7, 73.6)
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
Commit message: PCB work in progress
Parts:
- C1, C2, C3, C4, C5, C6, C7, D1, D10, D11, D12, D13, D14, D15, D16, D17, D18, D19, D2, D20, D21, D22, D23, D24, D25, D26, D27, D28, D29, D3, D30, D31, D32, D33, D34, D35, D36, D37, D38, D39, D4, D40, D41, D42, D43, D44, D45, D46, D47, D48, D49, D5, D50, D51, D52, D53, D54, D55, D56, D57, D58, D59, D6, D60, D61, D62, D63, D64, D65, D66, D67, D68, D7, D8, D9, R3, U1, Y1: moved to B.Cu
- MX58: footprint MX_Alps_Hybrid:MX-1.25U-NoLED -> MX_Alps_Hybrid:MX-2.25U-NoLED
- moved D5 370.0 mm to (54.8, 308.0), turned to 180 degrees
- moved D9 326.4 mm to (95.2, 288.9), turned to 180 degrees
- moved MX61 304.0 mm to (307.2, 263.5)
- moved MX1 302.2 mm to (52.4, 225.4)
- moved D19 293.9 mm to (133.3, 288.9), turned to 180 degrees
- moved D4 292.1 mm to (64.3, 288.9), turned to 180 degrees
- moved D29 286.4 mm to (171.4, 288.9), turned to 180 degrees
- moved D67 284.3 mm to (347.7, 231.8), turned to 180 degrees
- moved MX67 276.5 mm to (347.7, 225.4)
- moved MX40 274.8 mm to (309.6, 301.6)
- moved MX13 272.7 mm to (104.8, 263.5)
- moved MX35 271.6 mm to (288.1, 301.6)
- moved D34 267.9 mm to (190.5, 288.9), turned to 180 degrees
- moved MX30 263.5 mm to (264.3, 301.6)
- moved MX58 259.2 mm to (297.7, 282.6)
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Other:
- board outline added: 314.3 x 95.2 mm

Commit message: mocked up pcb
Parts:
- F1, R1, R2, R4, SW1, USB1: moved to B.Cu
- moved SW1 226.9 mm to (350.0, 254.0), turned to 180 degrees
- moved USB1 217.6 mm to (350.0, 232.8), turned to -90 degrees
- moved F1 182.2 mm to (343.7, 242.9), turned to 90 degrees
- moved R2 173.3 mm to (352.4, 242.9), turned to -90 degrees
- moved R4 155.3 mm to (356.4, 242.9), turned to 90 degrees
- moved R1 152.6 mm to (348.8, 242.9), turned to -90 degrees
- moved C6 22.5 mm to (335.8, 280.8)
- moved C7 22.5 mm to (343.5, 289.7)
- moved D56 22.5 mm to (288.1, 265.9)
- moved D61 22.5 mm to (323.9, 285.0)
- moved MX61 22.5 mm to (323.9, 278.6)
- moved R3 22.5 mm to (335.8, 276.7)
- moved MX56 22.5 mm to (288.1, 259.6)
- moved Y1 22.5 mm to (347.5, 268.5)
- moved D19 22.5 mm to (150.0, 304.0)
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
Commit message: changed pcb to work with unified daughterboard
Parts:
- removed USB1: Molex-0548190589, random-keyboard-parts:Molex-0548190589
- added J1: JST SH 4-pin, Connector_JST:JST_SH_SM04B-SRSS-TB_1x04-1MP_P1.00mm_Horizontal, B.Cu at (350.0, 253.2)
- added U2: SRV05-4, Package_TO_SOT_SMD:SOT-23-6, B.Cu at (341.3, 261.1)
- moved SW1 48.1 mm to (308.8, 278.6)
- moved R4 42.9 mm to (355.6, 285.8), turned to -90 degrees
- moved R1 19.1 mm to (347.7, 261.9)
- moved R2 19.1 mm to (351.6, 261.9), turned to 90 degrees
- moved F1 11.3 mm to (342.9, 254.2), turned to -90 degrees
Connections:
- F1 pad 1: VCC -> VBUS

Commit message: Working on traces
Parts:
- moved U2 11.3 mm to (349.9, 253.7)
- moved F1 9.41 mm to (344.0, 263.5)
- moved J1 6.35 mm to (350.0, 246.9)
- moved R1 5.37 mm to (352.0, 258.8)
- moved R2 4.51 mm to (348.4, 258.8), turned to -90 degrees
- moved D25 0.06 mm to (257.2, 323.1), turned to 0 degrees
- turned D2 to 0 degrees
- turned D1 to 0 degrees
- turned D10 to 0 degrees
- turned D11 to 0 degrees
- turned D12 to 0 degrees
- turned D13 to 0 degrees
- turned D14 to 0 degrees
- turned D15 to 0 degrees
- turned D16 to 0 degrees
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Connections:
- R1 pad 1: D + -> D+
- R2 pad 1: D - -> D-
Routing:
- net ROW0: track 0.00 -> 333.2 mm, vias 0 -> 28
- net ROW2: track 0.00 -> 327.4 mm, vias 0 -> 24
- net ROW1: track 0.00 -> 325.8 mm, vias 0 -> 26
- net ROW3: track 0.00 -> 313.7 mm, vias 0 -> 18
- net ROW4: track 0.00 -> 313.5 mm
- net COL9: track 0.00 -> 188.7 mm
- net COL6: track 0.00 -> 183.7 mm
- net COL8: track 0.00 -> 179.2 mm
- net COL7: track 0.00 -> 179.1 mm
- net COL5: track 0.00 -> 176.7 mm
- net COL4: track 0.00 -> 174.2 mm
- net COL3: track 0.00 -> 120.5 mm
- net GND: track 0.00 -> 97.4 mm, vias 0 -> 2
- net COL1: track 0.00 -> 95.8 mm
- net COL2: track 0.00 -> 94.3 mm
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
Commit message: finnished traces
Connections:
- U1 pad 1: unconnected-(U1-PE6) -> COL11
- U1 pad 10: unconnected-(U1-PB2) -> COL2
- U1 pad 11: unconnected-(U1-PB3) -> COL1
- U1 pad 12: unconnected-(U1-PB7) -> COL12
- U1 pad 18: unconnected-(U1-PD0) -> COL0
- U1 pad 21: unconnected-(U1-PD3) -> COL14
- U1 pad 22: unconnected-(U1-PD5) -> COL13
- U1 pad 25: unconnected-(U1-PD4) -> ROW0
- U1 pad 26: unconnected-(U1-PD6) -> ROW1
- U1 pad 27: unconnected-(U1-PD7) -> ROW2
- U1 pad 28: unconnected-(U1-PB4) -> ROW3
- U1 pad 29: unconnected-(U1-PB5) -> ROW4
- U1 pad 36: unconnected-(U1-PF7) -> COL5
- U1 pad 37: unconnected-(U1-PF6) -> COL6
- U1 pad 38: unconnected-(U1-PF5) -> COL7
- U1 pad 39: unconnected-(U1-PF4) -> COL8
- U1 pad 40: unconnected-(U1-PF1) -> COL9
- U1 pad 41: unconnected-(U1-PF0) -> COL10
- U1 pad 8: unconnected-(U1-PB0) -> COL4
- U1 pad 9: unconnected-(U1-PB1) -> COL3
Routing:
- net COL0: track 83.4 -> 412.1 mm, vias 0 -> 6
- net COL1: track 95.8 -> 399.5 mm, vias 0 -> 2
- net COL2: track 94.3 -> 375.7 mm, vias 0 -> 2
- net COL4: track 174.2 -> 377.6 mm, vias 0 -> 4
- net COL3: track 120.5 -> 320.1 mm, vias 0 -> 2
- net COL5: track 176.7 -> 286.5 mm, vias 0 -> 2
- net COL10: track 68.6 -> 148.1 mm, vias 0 -> 4
- net COL6: track 183.7 -> 259.7 mm, vias 0 -> 2
- net COL7: track 179.1 -> 237.6 mm, vias 0 -> 2
- net ROW4: track 313.5 -> 363.4 mm, vias 0 -> 2
- net ROW0: track 333.2 -> 379.2 mm, vias 28 -> 29
- net COL11: track 79.1 -> 117.2 mm, vias 0 -> 2
- net ROW3: track 313.7 -> 346.4 mm, vias 18 -> 20
- net COL8: track 179.2 -> 210.6 mm, vias 0 -> 2
- net COL9: track 188.7 -> 214.1 mm, vias 0 -> 4
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