File: PCB/keyboard.kicad_pcb (KiCad board)
At the start: 2 copper layers, 314.3 x 95.2 mm, 158 parts, among them J1 JST SH 4-pin, SW1 SW_Push, U1 ATmega32U4-A, U2 SRV05-4, Y1 16MHz

Commit message: redid wiring (again) no checks yet
Parts:
- added MX69: MX-NoLED, MX_Only:MXOnly-1.5U-NoLED, F.Cu at (73.8, 316.7)
- added MX70: MX-NoLED, MX_Only:MXOnly-1U-NoLED, F.Cu at (97.6, 316.7)
- added MX71: MX-NoLED, MX_Only:MXOnly-1.5U-NoLED, F.Cu at (121.4, 316.7)
- added MX72: MX-NoLED, MX_Only:MXOnly-7U-ReversedStabilizers-NoLED, F.Cu at (202.4, 316.7)
- added MX73: MX-NoLED, marbastlib-mx:SW_MX_1.75u_stp, F.Cu at (71.4, 278.6)
- added MX74: MX-NoLED, MX_Only:MXOnly-ISO-ReversedStabilizers-NoLED, F.Cu at (333.4, 269.1)
- added MX75: MX-NoLED, MX_Only:MXOnly-1U-NoLED, F.Cu at (311.9, 278.6)
- MX20: footprint MX_Only:MXOnly-6.25U-NoLED -> MX_Only:MXOnly-6.25U-ReversedStabilizers-NoLED
- moved C1 216.5 mm to (154.7, 322.1)
- moved C4 211.6 mm to (152.1, 314.2), turned to -90 degrees
- moved SW1 211.6 mm to (140.6, 314.1), turned to 90 degrees
- moved R3 210.1 mm to (157.8, 322.1), turned to -90 degrees
- moved C3 207.8 mm to (154.3, 310.6), turned to 0 degrees
- moved Y1 206.6 mm to (155.8, 314.1), turned to -90 degrees
- moved C5 199.9 mm to (154.8, 304.7), turned to 180 degrees
- moved C6 195.9 mm to (165.7, 322.9), turned to 0 degrees
- moved U1 187.6 mm to (165.8, 312.6), turned to 90 degrees
- moved F1 177.2 mm to (180.8, 311.5), turned to 180 degrees
- moved C7 175.1 mm to (174.3, 318.4), turned to 90 degrees
- moved R4 172.7 mm to (171.4, 304.8), turned to 0 degrees
- moved C2 168.1 mm to (173.9, 307.7), turned to -90 degrees
- moved R1 149.0 mm to (219.6, 316.7), turned to 180 degrees
- moved R2 145.6 mm to (219.6, 314.2), turned to 180 degrees
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Connections:
- U1 pad 1: ROW0 -> COL14
- U1 pad 10: ROW2 -> unconnected-(U1-PB2)
- U1 pad 11: ROW1 -> unconnected-(U1-PB3)
- U1 pad 12: COL14 -> unconnected-(U1-PB7)
- U1 pad 18: unconnected-(U1-PD0) -> ROW4
- U1 pad 19: unconnected-(U1-PD1) -> ROW0
- U1 pad 20: unconnected-(U1-PD2) -> ROW1
- U1 pad 21: unconnected-(U1-PD3) -> ROW2
- U1 pad 22: unconnected-(U1-PD5) -> ROW3
- U1 pad 31: COL6 -> COL7
- U1 pad 32: COL7 -> COL6
- U1 pad 8: ROW4 -> unconnected-(U1-PB0)
- U1 pad 9: ROW3 -> unconnected-(U1-PB1)
Routing:
- net ROW0: track 0.00 -> 478.0 mm
- net ROW2: track 0.00 -> 459.2 mm
- net ROW1: track 0.00 -> 457.6 mm
- net ROW4: track 0.13 -> 346.5 mm
- net ROW3: track 0.00 -> 337.6 mm, vias 0 -> 2
- net COL14: track 0.00 -> 288.5 mm, vias 0 -> 1
- net COL13: track 0.00 -> 283.0 mm, vias 0 -> 1
- net COL12: track 0.97 -> 248.5 mm, vias 0 -> 1
- net COL11: track 0.00 -> 216.9 mm, vias 0 -> 1
- net COL0: track 0.50 -> 196.2 mm
- net COL10: track 0.72 -> 193.4 mm, vias 0 -> 1
- net COL1: track 0.50 -> 176.3 mm, vias 0 -> 1
- net COL2: track 0.50 -> 169.6 mm, vias 0 -> 1
- net COL9: track 0.50 -> 169.4 mm, vias 0 -> 1
- net COL6: track 0.50 -> 159.5 mm
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- added copper zone on F.Cu, net GND

Commit message: still working on wiring
Routing:
- net D+: track 13.0 -> 13.7 mm
Changed lines of the file:
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@@
   (gr_arc (start 59.53125 232.56875) (mid 59.996218 231.446218) (end 61.11875 230.98125)
     (stroke (width 0.05) (type default)) (layer "Edge.Cuts"))
+  (gr_arc (start 373.85625 324.64375) (mid 373.391282 325.766282) (end 372.26875 326.23125)
+    (stroke (width 0.05) (type default)) (layer "Edge.Cuts"))
   (gr_line (start 59.53125 324.64375) (end 59.53125 232.56875)
-    (stroke (width 0.05) (type default)) (layer "Edge.Cuts"))
-  (gr_arc (start 373.85625 324.64375) (mid 373.391282 325.766282) (end 372.26875 326.23125)
     (stroke (width 0.05) (type default)) (layer "Edge.Cuts"))
   (gr_arc (start 61.11875 326.23125) (mid 59.996218 325.766282) (end 59.53125 324.64375)
@@
   (segment (start 170.5375 304.8) (end 170.5375 306.108) (width 0.25) (layer "B.Cu") (net 87))
   (segment (start 170.5375 306.108) (end 169.76675 306.87875) (width 0.25) (layer "B.Cu") (net 87))
+  (segment (start 226.756 317.278) (end 226.40552 317.278) (width 0.2) (layer "B.Cu") (net 91))
+  (segment (start 226.40552 317.278) (end 226.40552 316.616803) (width 0.2) (layer "B.Cu") (net 91))
+  (segment (start 221.864325 317.299028) (end 221.862603 317.299028) (width 0.2) (layer "B.Cu") (net 91))
+  (segment (start 221.262603 316.70075) (end 220.559 316.70075) (width 0.2) (layer "B.Cu") (net 91))
+  (segment (start 231.405001 316.328001) (end 227.705999 316.328001) (width 0.2) (layer "B.Cu") (net 91))
+  (segment (start 224.519803 316.35348) (end 223.595283 317.278) (width 0.2) (layer "B.Cu") (net 91))
+  (segment (start 221.264325 316.70075) (end 221.262603 316.70075) (width 0.2) (layer "B.Cu") (net 91))
+  (segment (start 226.142197 316.35348) (end 224.519803 316.35348) (width 0.2) (layer "B.Cu") (net 91))
+  (segment (start 227.705999 316.328001) (end 226.756 317.278) (width 0.2) (layer "B.Cu") (net 91))
   (segment (start 223.595283 317.278) (end 223.039853 317.278) (width 0.2) (layer "B.Cu") (net 91))
-  (segment (start 222.462603 316.70075) (end 220.559 316.70075) (width 0.2) (layer "B.Cu") (net 91))
-  (segment (start 226.142197 316.35348) (end 224.519803 316.35348) (width 0.2) (layer "B.Cu") (net 91))
-  (segment (start 226.40552 316.616803) (end 226.142197 316.35348) (width 0.2) (layer "B.Cu") (net 91))
-  (segment (start 231.405001 316.328001) (end 227.705999 316.328001) (width 0.2) (layer "B.Cu") (net 91))
-  (segment (start 226.756 317.278) (end 226.40552 317.278) (width 0.2) (layer "B.Cu") (net 91))
-  (segment (start 227.705999 316.328001) (end 226.756 317.278) (width 0.2) (layer "B.Cu") (net 91))
-  (segment (start 224.519803 316.35348) (end 223.595283 317.278) (width 0.2) (layer "B.Cu") (net 91))
-  (segment (start 226.40552 317.278) (end 226.40552 316.616803) (width 0.2) (layer "B.Cu") (net 91))
   (segment (start 231.68 316.603) (end 231.405001 316.328001) (width 0.2) (layer "B.Cu") (net 91))
   (segment (start 223.039853 317.278) (end 222.462603 316.70075) (width 0.2) (layer "B.Cu") (net 91))
+  (segment (start 226.40552 316.616803) (end 226.142197 316.35348) (width 0.2) (layer "B.Cu") (net 91))
+  (arc (start 221.862603 317.299028) (mid 221.65108 317.211412) (end 221.563464 316.999889) (width 0.2) (layer "B.Cu") (net 91))
+  (arc (start 222.462603 316.70075) (mid 222.25108 316.788366) (end 222.163464 316.999889) (width 0.2) (layer "B.Cu") (net 91))
+  (arc (start 221.563464 316.999889) (mid 221.475848 316.788366) (end 221.264325 316.70075) (width 0.2) (layer "B.Cu") (net 91))
+  (arc (start 222.163464 316.999889) (mid 222.075848 317.211412) (end 221.864325 317.299028) (width 0.2) (layer "B.Cu") (net 91))
   (segment (start 227.705999 315.877999) (end 226.756 314.928) (width 0.2) (layer "B.Cu") (net 92))
   (segment (start 224.33341 315.903489) (end 223.4089 316.827999) (width 0.2) (layer "B.Cu") (net 92))

Commit message: finnished implementing layouts
Routing:
- net ROW4: track 346.5 -> 343.4 mm
Changed lines of the file:
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@@
   (segment (start 177.8 300.1) (end 175.350489 302.549511) (width 0.25) (layer "B.Cu") (net 82))
   (segment (start 160.06675 308.57875) (end 160.06675 307.01227) (width 0.25) (layer "B.Cu") (net 82))
-  (segment (start 147.828 325.374) (end 233.807 325.374) (width 0.25) (layer "B.Cu") (net 83))
-  (segment (start 234.022771 325.589771) (end 237.528229 325.589771) (width 0.25) (layer "B.Cu") (net 83))
   (segment (start 159.231032 311.77875) (end 157.52844 310.076157) (width 0.25) (layer "B.Cu") (net 83))
+  (segment (start 208.28 321.183) (end 242.824 321.183) (width 0.25) (layer "B.Cu") (net 83))
   (segment (start 243.968 319.15) (end 244.475 319.15) (width 0.25) (layer "B.Cu") (net 83))
-  (segment (start 147.828 319.278) (end 147.828 325.374) (width 0.25) (layer "B.Cu") (net 83))
   (segment (start 152.278794 307.865277) (end 149.487597 305.07408) (width 0.25) (layer "B.Cu") (net 83))
+  (segment (start 147.7 319.15) (end 153.797 325.247) (width 0.25) (layer "B.Cu") (net 83))
   (segment (start 157.52844 310.076157) (end 157.52844 308.15044) (width 0.25) (layer "B.Cu") (net 83))
   (segment (start 157.5066 308.1286) (end 152.542116 308.1286) (width 0.25) (layer "B.Cu") (net 83))
-  (segment (start 130.175 319.15) (end 147.7 319.15) (width 0.25) (layer "B.Cu") (net 83))
+  (segment (start 169.30552 324.358) (end 205.105 324.358) (width 0.25) (layer "B.Cu") (net 83))
   (segment (start 149.487597 305.07408) (end 131.826 305.07408) (width 0.25) (layer "B.Cu") (net 83))
   (segment (start 152.542116 308.1286) (end 152.278794 307.865277) (width 0.25) (layer "B.Cu") (net 83))
+  (segment (start 168.41652 325.247) (end 169.30552 324.358) (width 0.25) (layer "B.Cu") (net 83))
   (segment (start 131.826 319.151) (end 131.825 319.15) (width 0.25) (layer "B.Cu") (net 83))
-  (segment (start 147.7 319.15) (end 147.828 319.278) (width 0.25) (layer "B.Cu") (net 83))
-  (segment (start 237.528229 325.589771) (end 243.968 319.15) (width 0.25) (layer "B.Cu") (net 83))
+  (segment (start 244.475 319.532) (end 244.475 319.15) (width 0.25) (layer "B.Cu") (net 83))
+  (segment (start 205.105 324.358) (end 208.28 321.183) (width 0.25) (layer "B.Cu") (net 83))
   (segment (start 131.826 305.07408) (end 131.826 319.151) (width 0.25) (layer "B.Cu") (net 83))
+  (segment (start 153.797 325.247) (end 168.41652 325.247) (width 0.25) (layer "B.Cu") (net 83))
   (segment (start 105.56875 319.15) (end 130.175 319.15) (width 0.25) (layer "B.Cu") (net 83))
+  (segment (start 242.824 321.183) (end 244.475 319.532) (width 0.25) (layer "B.Cu") (net 83))
   (segment (start 157.52844 308.15044) (end 157.5066 308.1286) (width 0.25) (layer "B.Cu") (net 83))
   (segment (start 372.26875 319.15) (end 244.475 319.15) (width 0.25) (layer "B.Cu") (net 83))
   (segment (start 82.55 319.15) (end 105.56875 319.15) (width 0.25) (layer "B.Cu") (net 83))
   (segment (start 160.06675 311.77875) (end 159.231032 311.77875) (width 0.25) (layer "B.Cu") (net 83))
+  (segment (start 130.175 319.15) (end 147.7 319.15) (width 0.25) (layer "B.Cu") (net 83))
   (segment (start 131.825 319.15) (end 130.175 319.15) (width 0.25) (layer "B.Cu") (net 83))
-  (segment (start 233.807 325.374) (end 234.022771 325.589771) (width 0.25) (layer "B.Cu") (net 83))
   (segment (start 369.15725 235.42625) (end 372.237 238.506) (width 0.25) (layer "B.Cu") (net 84))
   (segment (start 372.237 238.506) (end 372.237 239.65) (width 0.25) (layer "B.Cu") (net 84))

Commit message: relocated JST
Parts:
- moved R1 68.2 mm to (227.1, 248.9)
- moved J1 68.2 mm to (241.1, 248.3)
- moved R2 68.2 mm to (227.1, 246.4)
- moved U2 68.2 mm to (233.2, 248.3)
Connections:
- R1 pad 2: Net-(U1-D+) -> D+
- R2 pad 2: Net-(U1-D-) -> D-
- U1 pad 3: Net-(U1-D-) -> D-
- U1 pad 4: Net-(U1-D+) -> D+
Routing:
- net D+: track 13.7 -> 152.5 mm
- net D-: track 13.7 -> 152.5 mm
- net VBUS: track 53.7 -> 130.5 mm
- net Net-(U1-D+): track 59.0 -> 0.00 mm
- net Net-(U1-D-): track 58.3 -> 0.00 mm
- net COL14: track 288.5 -> 291.4 mm, vias 1 -> 3
- net COL13: track 283.0 -> 285.3 mm, vias 1 -> 3
- net COL12: track 248.5 -> 250.4 mm, vias 1 -> 3
- net COL11: track 216.9 -> 218.3 mm, vias 1 -> 3
- net COL10: track 193.4 -> 194.3 mm, vias 1 -> 3
- net ROW2: track 459.2 -> 460.0 mm, vias 0 -> 2
- net ROW3: track 337.6 -> 338.1 mm, vias 2 -> 4
- net COL9: track 169.4 -> 169.9 mm, vias 1 -> 3
- net ROW1: track 457.6 -> 457.9 mm, vias 0 -> 2
- net GND: track 82.5 -> 82.1 mm, vias 22 -> 26
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