File: PCB/keyboard.kicad_sch (KiCad schematic)
At the start: 153 parts, among them J1 JST SH 4-pin, SW1 SW_Push, U1 ATmega32U4-A, U2 SRV05-4, Y1 16MHz

Commit message: started reworking wiring (again), only mx footprints now
Parts:
- MX1, MX10, MX11, MX12, MX13, MX14, MX16, MX17, MX18, MX19, MX21, MX22, MX23, MX24, MX26, MX27, MX28, MX29, MX31, MX32, MX33, MX34, MX36, MX37, MX38, MX39, MX40, MX41, MX42, MX43, MX44, MX45, MX46, MX47, MX48, MX49, MX50, MX51, MX52, MX53, MX54, MX55, MX56, MX57, MX59, MX6, MX60, MX62, MX65, MX66, MX67, MX68, MX7, MX8, MX9: footprint MX_Alps_Hybrid:MX-1U-NoLED -> MX_Only:MXOnly-1U-NoLED
- MX15, MX25, MX30, MX35, MX5: footprint MX_Alps_Hybrid:MX-1.25U-NoLED -> MX_Only:MXOnly-1.25U-NoLED
- MX2, MX64: footprint MX_Alps_Hybrid:MX-1.5U-NoLED -> MX_Only:MXOnly-1.5U-NoLED
- MX20: footprint MX_Alps_Hybrid:MX-6.25U-NoLED -> MX_Only:MXOnly-6.25U-NoLED
- MX3: footprint MX_Alps_Hybrid:MX-1.75U-NoLED -> MX_Only:MXOnly-1.75U-NoLED
- MX4, MX58, MX61: footprint MX_Alps_Hybrid:MX-2.25U-NoLED -> MX_Only:MXOnly-2.25U-NoLED
- MX63: footprint MX_Alps_Hybrid:MX-2U-NoLED -> MX_Only:MXOnly-2U-NoLED

Commit message: redid wiring (again) no checks yet
Parts:
- added MX69, MX71: MX-NoLED, MX_Only:MXOnly-1.5U-NoLED, symbol MX_Alps_Hybrid:MX-NoLED
- added MX70, MX75: MX-NoLED, MX_Only:MXOnly-1U-NoLED, symbol MX_Alps_Hybrid:MX-NoLED
- added MX72: MX-NoLED, MX_Only:MXOnly-7U-ReversedStabilizers-NoLED, symbol MX_Alps_Hybrid:MX-NoLED
- added MX73: MX-NoLED, marbastlib-mx:SW_MX_1.75u_stp, symbol MX_Alps_Hybrid:MX-NoLED
- added MX74: MX-NoLED, MX_Only:MXOnly-ISO-ReversedStabilizers-NoLED, symbol MX_Alps_Hybrid:MX-NoLED
- MX20: footprint MX_Only:MXOnly-6.25U-NoLED -> MX_Only:MXOnly-6.25U-ReversedStabilizers-NoLED
Connections:
- net COL0: now also MX69.1 (COL), MX73.1 (COL)
- net COL1: now also MX70.1 (COL)
- net COL13: now also MX74.1 (COL), MX75.1 (COL)
- net COL14: now also U1.1 (PE6); no longer U1.12 (PB7)
- net COL2: now also MX71.1 (COL)
- net COL6: now also U1.32 (PC7), MX72.1 (COL); no longer U1.31 (PC6)
- net COL7: now also U1.31 (PC6); no longer U1.32 (PC7)
- net ROW0: now also U1.19 (PD1); no longer U1.1 (PE6)
- net ROW1: now also U1.20 (PD2); no longer U1.11 (PB3)
- net ROW2: now also U1.21 (PD3); no longer U1.10 (PB2)
- net ROW3: now also U1.22 (PD5); no longer U1.9 (PB1)
- net ROW4: now also U1.18 (PD0); no longer U1.8 (PB0)
- net at D20.2 (A), MX20.2 (ROW): now also MX72.2 (ROW)
- net at D61.2 (A), MX61.2 (ROW): now also MX74.2 (ROW)
- net at D64.2 (A), MX64.2 (ROW): now also MX75.2 (ROW)
- net at D10.2 (A), MX10.2 (ROW): now also MX70.2 (ROW)
- net at D15.2 (A), MX15.2 (ROW): now also MX71.2 (ROW)
- net at D3.2 (A), MX3.2 (ROW): now also MX73.2 (ROW)
- net at D5.2 (A), MX5.2 (ROW): now also MX69.2 (ROW)
